File: i2c 24vout/i2c 24vout.kicad_pcb (KiCad board)
At the start: 2 copper layers, 123.2 x 50.2 mm, 97 parts, among them J1 power in, J10 Conn_01x01, J2 Conn_01x04, J3 Conn_01x04, J4 Conn_01x04, J5 Conn_01x04, J6 to qwiic breakout, J7 qwiic 1, J8 qwiic 2, J9 Conn_01x01, U1 ILQ620GB-X009, U2 ILQ620GB-X009, U3 ILQ620GB-X009, U4 ILQ620GB-X009, U5 PCA9685PW

Commit message: DFM 24vout
Parts:
- C1, C10, C11, C12, C13, C14, C15, C16, C2, C3, C4, C5, C6, C7, C8, C9, R17, R18, R19, R20, R21, R22, R23, R24, R25, R26, R27, R28, R29, R30, R31, R32: moved to F.Cu
- moved R4 12.6 mm to (111.9, 100.5), turned to 90 degrees
- moved R3 9.28 mm to (110.4, 100.8), turned to 90 degrees
- moved R2 6.00 mm to (108.8, 101.3), turned to 90 degrees
- moved R7 4.06 mm to (142.1, 101.1), turned to 90 degrees
- moved R1 3.94 mm to (107.3, 101.3), turned to 90 degrees
- moved R32 3.50 mm to (191.5, 118.7), turned to 0 degrees
- moved C15 3.49 mm to (186.4, 117.1), turned to 0 degrees
- moved R31 3.49 mm to (186.4, 118.7), turned to 0 degrees
- moved C12 3.49 mm to (168.9, 117.1), turned to 0 degrees
- moved C13 3.49 mm to (176.4, 117.1), turned to 0 degrees
- moved C14 3.49 mm to (181.5, 117.1), turned to 0 degrees
- moved C5 3.49 mm to (131.2, 117.0), turned to 0 degrees
- moved C9 3.49 mm to (153.8, 117.1), turned to 0 degrees
- moved R21 3.49 mm to (131.2, 118.6), turned to 0 degrees
- moved R25 3.49 mm to (153.8, 118.7), turned to 0 degrees
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Routing:
- net GND: track 15.0 -> 158.4 mm
- net /pwm3: track 19.7 -> 5.70 mm
- net Net-(R4-Pad1): track 2.22 -> 13.8 mm
- net /pwm2: track 16.5 -> 8.09 mm
- net Net-(R3-Pad1): track 2.17 -> 10.2 mm
- net VCC: track 66.4 -> 73.2 mm
- net Net-(R2-Pad1): track 2.17 -> 6.59 mm
- net /pwm6: track 32.0 -> 28.1 mm, vias 0 -> 2
- net /pwm1: track 14.3 -> 10.7 mm
- net Net-(J3-Pin_2): track 7.83 -> 10.9 mm
- net Net-(J5-Pin_4): track 7.63 -> 10.7 mm
- net Net-(J5-Pin_3): track 7.67 -> 10.7 mm
- net Net-(J5-Pin_2): track 7.65 -> 10.7 mm
- net Net-(J5-Pin_1): track 7.68 -> 10.8 mm
- net Net-(J4-Pin_4): track 7.63 -> 10.7 mm
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